Commit message: oprava nacitani mapy

File: description/robot.urdf.xacro (robot description, xacro)
@@ -5,5 +5,5 @@
     <!-- <xacro:include filename="ros2_control.xacro"/> -->
     <xacro:include filename="lidar.xacro"/>
-    <xacro:include filename="camera.xacro"/>
-    <!-- <xacro:include filename="depth_camera.xacro"/> -->
+    <!--<xacro:include filename="camera.xacro"/> -->
+    <xacro:include filename="depth_camera.xacro"/>
 </robot>

File: description/robot_core.xacro (robot description, xacro)
@@ -22,4 +22,12 @@
     <!-- BASE LINK -->
     <link name="base_link">
+    </link>
+    <!-- BASE_FOOTPRINT LINK -->
+    <joint name="base_footprint_joint" type="fixed">
+        <parent link="base_link"/>
+        <child link="base_footprint"/>
+        <origin xyz="0 0 0" rpy="0 0 0"/>
+    </joint>
+    <link name="base_footprint">
     </link>
     <!-- CHASSIS LINK -->

File: install/articubot_one/share/articubot_one/description/camera.xacro (robot description, xacro)
@@ -1 +1 @@
-/home/dominikfink/dev_ws/articubot_one/description/camera.xacro
+/home/dominikfink/dev_ws/src/articubot_one/description/camera.xacro

File: install/articubot_one/share/articubot_one/description/gazebo_control.xacro (robot description, xacro)
@@ -1 +1 @@
-/home/dominikfink/dev_ws/articubot_one/description/gazebo_control.xacro
+/home/dominikfink/dev_ws/src/articubot_one/description/gazebo_control.xacro

File: install/articubot_one/share/articubot_one/description/inertial_macros.xacro (robot description, xacro)
@@ -1 +1 @@
-/home/dominikfink/dev_ws/articubot_one/description/inertial_macros.xacro
+/home/dominikfink/dev_ws/src/articubot_one/description/inertial_macros.xacro

File: install/articubot_one/share/articubot_one/description/lidar.xacro (robot description, xacro)
@@ -1 +1 @@
-/home/dominikfink/dev_ws/articubot_one/description/lidar.xacro
+/home/dominikfink/dev_ws/src/articubot_one/description/lidar.xacro

File: install/articubot_one/share/articubot_one/description/robot.urdf.xacro (robot description, xacro)
@@ -1 +1 @@
-/home/dominikfink/dev_ws/articubot_one/description/robot.urdf.xacro
+/home/dominikfink/dev_ws/src/articubot_one/description/robot.urdf.xacro

File: install/articubot_one/share/articubot_one/description/robot_core.xacro (robot description, xacro)
@@ -1 +1 @@
-/home/dominikfink/dev_ws/articubot_one/description/robot_core.xacro
+/home/dominikfink/dev_ws/src/articubot_one/description/robot_core.xacro
