Commit message: jazzy update + new maps

File: description/depth_camera.xacro (robot description, xacro)
@@ -1,4 +1,7 @@
 <?xml version="1.0"?>
-<robot xmlns:xacro="http://www.ros.org/wiki/xacro" >
+<robot xmlns:xacro="http://www.ros.org/wiki/xacro">
+    <!-- definice pi pro rpy -->
+    <xacro:property name="pi" value="3.14159265359"/>
+    <!-- camera joint -->
     <joint name="camera_joint" type="fixed">
         <parent link="chassis"/>
@@ -6,4 +9,5 @@
         <origin xyz="0.305 0 0.08" rpy="0 0 0"/>
     </joint>
+    <!-- camera link -->
     <link name="camera_link">
         <visual>
@@ -14,4 +18,5 @@
         </visual>
     </link>
+    <!-- optical joint -->
     <joint name="camera_optical_joint" type="fixed">
         <parent link="camera_link"/>
@@ -19,5 +24,6 @@
         <origin xyz="0 0 0" rpy="${-pi/2} 0 ${-pi/2}"/>
     </joint>
-    <link name="camera_link_optical"></link>
+    <link name="camera_link_optical"/>
+    <!-- Gazebo sensor -->
     <gazebo reference="camera_link">
         <material>Gazebo/Red</material>
@@ -29,5 +35,5 @@
                 <horizontal_fov>1.089</horizontal_fov>
                 <image>
-                    <format>B8G8R8</format>
+                    <format>R8G8B8</format>
                     <width>640</width>
                     <height>480</height>
@@ -38,8 +44,14 @@
                 </clip>
             </camera>
-            <plugin name="camera_controller" filename="libgazebo_ros_camera.so">
+            <plugin name="camera_controller" filename="libgazebo_ros_depth_camera.so">
+                <ros>
+                    <namespace>/camera</namespace>
+                </ros>
+                <camera_name>camera</camera_name>
                 <frame_name>camera_link_optical</frame_name>
-                <min_depth>0.1</min_depth>
-                <max_depth>100.0</max_depth>
+                <update_rate>10.0</update_rate>
+                <depth_image_topic>depth/image_raw</depth_image_topic>
+                <depth_camera_info_topic>depth/camera_info</depth_camera_info_topic>
+                <point_cloud_topic>depth/points</point_cloud_topic>
             </plugin>
         </sensor>

Commit message: depth camera fix

File: description/depth_camera.xacro (robot description, xacro)
@@ -22,14 +22,15 @@
         <parent link="camera_link"/>
         <child link="camera_link_optical"/>
-        <origin xyz="0 0 0" rpy="${-pi/2} 0 ${-pi/2}"/>
+        <origin xyz="0 0 0" rpy="0 0 0"/>
     </joint>
     <link name="camera_link_optical"/>
-    <!-- Gazebo sensor -->
-    <gazebo reference="camera_link">
+    <!-- Gazebo Jetty sensor -->
+    <gazebo reference="camera_link_optical">
         <material>Gazebo/Red</material>
-        <sensor name="camera" type="depth">
+        <sensor name="depth_camera" type="depth">
             <pose>0 0 0 0 0 0</pose>
             <visualize>true</visualize>
             <update_rate>10</update_rate>
+            <always_on>true</always_on>
             <camera>
                 <horizontal_fov>1.089</horizontal_fov>
@@ -44,15 +45,7 @@
                 </clip>
             </camera>
-            <plugin name="camera_controller" filename="libgazebo_ros_depth_camera.so">
-                <ros>
-                    <namespace>/camera</namespace>
-                </ros>
-                <camera_name>camera</camera_name>
-                <frame_name>camera_link_optical</frame_name>
-                <update_rate>10.0</update_rate>
-                <depth_image_topic>depth/image_raw</depth_image_topic>
-                <depth_camera_info_topic>depth/camera_info</depth_camera_info_topic>
-                <point_cloud_topic>depth/points</point_cloud_topic>
-            </plugin>
+            <topic>camera/depth</topic>
+            <!-- DŮLEŽITÉ: Gazebo bude používat stejný frame jako link -->
+            <gz_frame_id>camera_link_optical</gz_frame_id>
         </sensor>
     </gazebo>

File: description/robot.urdf.xacro (robot description, xacro)
@@ -5,5 +5,5 @@
      <!-- <xacro:include filename="ros2_control.xacro"/> -->
     <xacro:include filename="lidar.xacro"/>
-    <xacro:include filename="camera.xacro"/>
-    <!--<xacro:include filename="depth_camera.xacro"/> -->
+    <!-- <xacro:include filename="camera.xacro"/> -->
+    <xacro:include filename="depth_camera.xacro"/>
 </robot>

Commit message: obě kamery současně
depth bez obrazu, zkusit převod z pc na image?

File: description/depth_camera.xacro (robot description, xacro)
@@ -3,12 +3,12 @@
     <!-- definice pi pro rpy -->
     <xacro:property name="pi" value="3.14159265359"/>
-    <!-- camera joint -->
-    <joint name="camera_joint" type="fixed">
+    <!-- depth camera joint -->
+    <joint name="depth_camera_joint" type="fixed">
         <parent link="chassis"/>
-        <child link="camera_link"/>
+        <child link="depth_camera_link"/>
         <origin xyz="0.305 0 0.08" rpy="0 0 0"/>
     </joint>
-    <!-- camera link -->
-    <link name="camera_link">
+    <!-- depth camera link -->
+    <link name="depth_camera_link">
         <visual>
             <geometry>
@@ -18,13 +18,13 @@
         </visual>
     </link>
-    <!-- optical joint -->
-    <joint name="camera_optical_joint" type="fixed">
-        <parent link="camera_link"/>
-        <child link="camera_link_optical"/>
+    <!-- depth_camera optical joint -->
+    <joint name="depth_camera_optical_joint" type="fixed">
+        <parent link="depth_camera_link"/>
+        <child link="depth_camera_link_optical"/>
         <origin xyz="0 0 0" rpy="0 0 0"/>
     </joint>
-    <link name="camera_link_optical"/>
+    <link name="depth_camera_link_optical"/>
     <!-- Gazebo Jetty sensor -->
-    <gazebo reference="camera_link_optical">
+    <gazebo reference="depth_camera_link_optical">
         <material>Gazebo/Red</material>
         <sensor name="depth_camera" type="depth">
@@ -45,7 +45,7 @@
                 </clip>
             </camera>
-            <topic>camera/depth</topic>
+            <topic>depth_camera/depth</topic>
             <!-- DŮLEŽITÉ: Gazebo bude používat stejný frame jako link -->
-            <gz_frame_id>camera_link_optical</gz_frame_id>
+            <gz_frame_id>depth_camera_link_optical</gz_frame_id>
         </sensor>
     </gazebo>

File: description/rgb_camera.xacro (robot description, xacro)
@@ -1,10 +1,10 @@
 <?xml version="1.0"?>
 <robot xmlns:xacro="http://www.ros.org/wiki/xacro" >
-    <joint name="camera_joint" type="fixed">
+    <joint name="rgb_camera_joint" type="fixed">
         <parent link="chassis"/>
-        <child link="camera_link"/>
+        <child link="rgb_camera_link"/>
         <origin xyz="0.276 0 0.181" rpy="0 0.18 0"/>
     </joint>
-    <link name="camera_link">
+    <link name="rgb_camera_link">
         <visual>
             <geometry>
@@ -21,18 +21,18 @@
         </visual>
     </link>
-    <joint name="camera_optical_joint" type="fixed">
-        <parent link="camera_link"/>
-        <child link="camera_link_optical"/>
+    <joint name="rgb_camera_optical_joint" type="fixed">
+        <parent link="rgb_camera_link"/>
+        <child link="rgb_camera_link_optical"/>
         <origin xyz="0 0 0" rpy="${-pi/2} 0 ${-pi/2}"/>
     </joint>
-    <link name="camera_link_optical"></link>
-    <gazebo reference="camera_link">
+    <link name="rgb_camera_link_optical"></link>
+    <gazebo reference="rgb_camera_link">
         <material>Gazebo/Black</material>
-        <sensor name="camera" type="camera">
+        <sensor name="rgb_camera" type="camera">
             <pose> 0 0 0 0 0 0 </pose>
             <visualize>true</visualize>
             <update_rate>10</update_rate>
             <camera>
-                <camera_info_topic>camera/camera_info</camera_info_topic>
+                <camera_info_topic>rgb_camera/camera_info</camera_info_topic>
                 <horizontal_fov>1.089</horizontal_fov>
                 <image>
@@ -46,6 +46,6 @@
                 </clip>
             </camera>
-            <topic>camera/image_raw</topic>
-            <gz_frame_id>camera_link_optical</gz_frame_id>
+            <topic>rgb_camera/image_raw</topic>
+            <gz_frame_id>rgb_camera_link_optical</gz_frame_id>
         </sensor>
     </gazebo>

File: description/robot.urdf.xacro (robot description, xacro)
@@ -5,5 +5,5 @@
      <!-- <xacro:include filename="ros2_control.xacro"/> -->
     <xacro:include filename="lidar.xacro"/>
-    <!-- <xacro:include filename="camera.xacro"/> -->
+    <xacro:include filename="rgb_camera.xacro"/>
     <xacro:include filename="depth_camera.xacro"/>
 </robot>
